File: hardware/radio_dev_board/USB_Serial.sch (KiCad schematic (older format))
At the start: 13 parts, among them J1 USB_C_Receptacle_USB2.0V1, U1 FT232RL

Commit message: added program and misc buttons. Finish layout
Parts:
- removed C4, C5, C7: 0.1, Capacitor_SMD:C_0603_1608Metric_Pad1.05x0.95mm_HandSolder, symbol Device:C
- removed R5: 1K, Resistor_SMD:R_0603_1608Metric_Pad1.05x0.95mm_HandSolder, symbol Device:R
- removed U1: FT232RL, Package_SO:SSOP-28_5.3x10.2mm_P0.65mm, symbol Interface_USB:FT232RL
- added C28, C29, C31: 0.1, Capacitor_SMD:C_0603_1608Metric_Pad1.05x0.95mm_HandSolder, symbol Device:C
- added R26: 1K, Resistor_SMD:R_0603_1608Metric_Pad1.05x0.95mm_HandSolder, symbol Device:R
- added SW2: SW_Push, Button_Switch_SMD:SW_SPST_PTS645, symbol Switch:SW_Push
- added U11: FT232RL, Package_SO:SSOP-28_5.3x10.2mm_P0.65mm, symbol Interface_USB:FT232RL
- renumbered C3 to C27, C6 to C30, D3 to D13, D4 to D14, J1 to J6, R2 to R23, R3 to R24, R4 to R25
Connections:
- net +5V: now also C29.1, U11.19 (~RESET~), U11.20 (VCC), U11.4 (VCCIO)
- net GND: now also C28.2, C29.2, SW2.2, U11.18 (GND), U11.21 (GND), U11.25 (AGND), U11.7 (GND)
- net TX: now also R26.1
- net ~Reset: now also C31.1, SW2.1
- net at R25.2: now also U11.1 (TXD)
- net at J6.A6 (D+), J6.B6 (D+): now also U11.15 (USBD+)
- net at J6.A7 (D-), J6.B7 (D-): now also U11.16 (USBD-)
- net at R24.1: now also U11.22 (CBUS1)
- net at R23.1: now also U11.23 (CBUS0)
- new net: C28.1, U11.17 (3V3OUT)
- new net: C31.2, U11.2 (DTR)
- new net: R26.2, U11.5 (RXD)
Changed lines of the file:
@@
 $EndDescr
 $Comp
-L power:GND #PWR011
+L power:GND #PWR079
 U 1 1 5D71ECE6
 P 4900 5550
-F 0 "#PWR011" H 4900 5300 50  0001 C CNN
+F 0 "#PWR079" H 4900 5300 50  0001 C CNN
 F 1 "GND" H 4905 5377 50  0000 C CNN
 F 2 "" H 4900 5550 50  0001 C CNN
@@
 $EndComp
 $Comp
-L Device:C C3
+L Device:C C27
 U 1 1 5D71EF5D
 P 4900 4200
-F 0 "C3" H 5015 4246 50  0000 L CNN
+F 0 "C27" H 5015 4246 50  0000 L CNN
 F 1 "0.01" H 5015 4155 50  0000 L CNN
 F 2 "Capacitor_SMD:C_0603_1608Metric_Pad1.05x0.95mm_HandSolder" H 4938 4050 50  0001 C CNN
@@
 $EndComp
 $Comp
-L Interface_USB:FT232RL U1
-U 1 1 5D71F5F1
+L Interface_USB:FT232RL U11
+U 1 1 5E0B10D6
 P 6300 4100
-F 0 "U1" H 6300 5281 50  0000 C CNN
+F 0 "U11" H 6300 5281 50  0000 C CNN
 F 1 "FT232RL" H 6300 5190 50  0000 C CNN
 F 2 "Package_SO:SSOP-28_5.3x10.2mm_P0.65mm" H 6300 4100 50  0001 C CNN
@@
 $EndComp
 $Comp
-L Device:C C4
-U 1 1 5D720B59
+L Device:C C28
+U 1 1 5E0B10D7
 P 5250 5200
-F 0 "C4" H 5365 5246 50  0000 L CNN
+F 0 "C28" H 5365 5246 50  0000 L CNN
 F 1 "0.1" H 5365 5155 50  0000 L CNN
 F 2 "Capacitor_SMD:C_0603_1608Metric_Pad1.05x0.95mm_HandSolder" H 5288 5050 50  0001 C CNN
@@
 $EndComp
 $Comp
-L Device:C C5
-U 1 1 5D72111C
+L Device:C C29
+U 1 1 5E0B10D8
 P 5650 5200
-F 0 "C5" H 5765 5246 50  0000 L CNN
+F 0 "C29" H 5765 5246 50  0000 L CNN
 F 1 "0.1" H 5765 5155 50  0000 L CNN
 F 2 "Capacitor_SMD:C_0603_1608Metric_Pad1.05x0.95mm_HandSolder" H 5688 5050 50  0001 C CNN
@@
 $EndComp
 $Comp
-L Device:R R4
+L Device:R R25
 U 1 1 5D721396
 P 8200 3400
-F 0 "R4" V 7993 3400 50  0000 C CNN
+F 0 "R25" V 7993 3400 50  0000 C CNN
 F 1 "1K" V 8084 3400 50  0000 C CNN
 F 2 "Resistor_SMD:R_0603_1608Metric_Pad1.05x0.95mm_HandSolder" V 8130 3400 50  0001 C CNN
@@
 $EndComp
 $Comp
-L Device:LED D3
+L Device:LED D13
 U 1 1 5D721F76
 P 7450 2200
-F 0 "D3" V 7489 2083 50  0000 R CNN
+F 0 "D13" V 7489 2083 50  0000 R CNN
 F 1 "RX" V 7398 2083 50  0000 R CNN
 F 2 "LED_SMD:LED_0603_1608Metric_Pad1.05x0.95mm_HandSolder" H 7450 2200 50  0001 C CNN
@@
 $EndComp
 $Comp
-L Device:R R2
+L Device:R R23
 U 1 1 5D722822
 P 7450 2700
-F 0 "R2" H 7380 2654 50  0000 R CNN
+F 0 "R23" H 7380 2654 50  0000 R CNN
 F 1 "1K" H 7380 2745 50  0000 R CNN
 F 2 "Resistor_SMD:R_0603_1608Metric_Pad1.05x0.95mm_HandSolder" V 7380 2700 50  0001 C CNN
@@
 $EndComp
 $Comp
-L Device:LED D4
+L Device:LED D14
 U 1 1 5D723070
 P 7800 2200
-F 0 "D4" V 7839 2083 50  0000 R CNN
+F 0 "D14" V 7839 2083 50  0000 R CNN
 F 1 "TX" V 7748 2083 50  0000 R CNN
 F 2 "LED_SMD:LED_0603_1608Metric_Pad1.05x0.95mm_HandSolder" H 7800 2200 50  0001 C CNN
@@
 $EndComp
 $Comp
-L Device:R R3
+L Device:R R24
 U 1 1 5D722DD5
 P 7800 2700
-F 0 "R3" H 7730 2654 50  0000 R CNN
+F 0 "R24" H 7730 2654 50  0000 R CNN
 F 1 "1K" H 7730 2745 50  0000 R CNN
 F 2 "Resistor_SMD:R_0603_1608Metric_Pad1.05x0.95mm_HandSolder" V 7730 2700 50  0001 C CNN
@@
 $EndComp
 $Comp
-L Device:C C6
+L Device:C C30
 U 1 1 5D732335
 P 5950 2600
-F 0 "C6" H 6065 2646 50  0000 L CNN
+F 0 "C30" H 6065 2646 50  0000 L CNN
 F 1 "0.1" H 6065 2555 50  0000 L CNN
 F 2 "Capacitor_SMD:C_0603_1608Metric_Pad1.05x0.95mm_HandSolder" H 5988 2450 50  0001 C CNN
@@
 $EndComp
 $Comp
-L power:GND #PWR013
+L power:GND #PWR081
 U 1 1 5D742392
 P 5650 5550
-F 0 "#PWR013" H 5650 5300 50  0001 C CNN
+F 0 "#PWR081" H 5650 5300 50  0001 C CNN
 F 1 "GND" H 5655 5377 50  0000 C CNN
 F 2 "" H 5650 5550 50  0001 C CNN
@@
 $EndComp
 $Comp
-L power:GND #PWR012
-U 1 1 5D74282F
+L power:GND #PWR080
+U 1 1 5E0B10E0
 P 5250 5550
-F 0 "#PWR012" H 5250 5300 50  0001 C CNN
+F 0 "#PWR080" H 5250 5300 50  0001 C CNN
 F 1 "GND" H 5255 5377 50  0000 C CNN
 F 2 "" H 5250 5550 50  0001 C CNN
@@
 $EndComp
 $Comp
-L power:+5V #PWR016
-U 1 1 5D75081A
+L power:+5V #PWR084
+U 1 1 5E0B10E1
 P 6250 1850
-F 0 "#PWR016" H 6250 1700 50  0001 C CNN
+F 0 "#PWR084" H 6250 1700 50  0001 C CNN
 F 1 "+5V" H 6265 2023 50  0000 C CNN
 F 2 "" H 6250 1850 50  0001 C CNN
@@
 $EndComp
 $Comp
-L power:+5V #PWR018
-U 1 1 5D750CFA
+L power:+5V #PWR086
+U 1 1 5E0B10E2
 P 7450 1800
-F 0 "#PWR018" H 7450 1650 50  0001 C CNN
+F 0 "#PWR086" H 7450 1650 50  0001 C CNN
 F 1 "+5V" H 7465 1973 50  0000 C CNN
 F 2 "" H 7450 1800 50  0001 C CNN
@@
 $EndComp
 $Comp
-L power:+5V #PWR019
-U 1 1 5D751062
+L power:+5V #PWR087
+U 1 1 5E0B10E3
 P 7800 1800
-F 0 "#PWR019" H 7800 1650 50  0001 C CNN
+F 0 "#PWR087" H 7800 1650 50  0001 C CNN
 F 1 "+5V" H 7815 1973 50  0000 C CNN
 F 2 "" H 7800 1800 50  0001 C CNN
@@
 $EndComp
 $Comp
-L power:GND #PWR017
-U 1 1 5D7525B9
+L power:GND #PWR085
+U 1 1 5E0B10E4
 P 6400 5550
-F 0 "#PWR017" H 6400 5300 50  0001 C CNN
+F 0 "#PWR085" H 6400 5300 50  0001 C CNN
 F 1 "GND" H 6405 5377 50  0000 C CNN
 F 2 "" H 6400 5550 50  0001 C CNN
@@
 $EndComp
 $Comp
-L power:GND #PWR015
+L power:GND #PWR083
 U 1 1 5D752BD0
 P 6100 5550
-F 0 "#PWR015" H 6100 5300 50  0001 C CNN
+F 0 "#PWR083" H 6100 5300 50  0001 C CNN
 F 1 "GND" H 6105 5377 50  0000 C CNN
 F 2 "" H 6100 5550 50  0001 C CNN
@@
 $EndComp
 $Comp
-L Device:R R5
-U 1 1 5D75D181
+L Device:R R26
+U 1 1 5E0B10E6
 P 8500 3500
-F 0 "R5" V 8293 3500 50  0000 C CNN
+F 0 "R26" V 8293 3500 50  0000 C CNN
 F 1 "1K" V 8384 3500 50  0000 C CNN
 F 2 "Resistor_SMD:R_0603_1608Metric_Pad1.05x0.95mm_HandSolder" V 8430 3500 50  0001 C CNN
@@
 $EndComp
 $Comp
-L Device:C C7
-U 1 1 5D75D707
+L Device:C C31
+U 1 1 5E0B10E7
 P 8200 3800
-F 0 "C7" V 7948 3800 50  0000 C CNN
+F 0 "C31" V 7948 3800 50  0000 C CNN
 F 1 "0.1" V 8039 3800 50  0000 C CNN
 F 2 "Capacitor_SMD:C_0603_1608Metric_Pad1.05x0.95mm_HandSolder" H 8238 3650 50  0001 C CNN
@@
 	7100 3800 8050 3800
 Wire Wire Line
-	8350 3800 8950 3800
+	8350 3800 9250 3800
 Wire Wire Line
 	4900 5550 4900 4350
@@
 	6250 2300 6250 2850
 $Comp
-L power:GND #PWR014
-U 1 1 5D78E49D
+L power:GND #PWR082
+U 1 1 5E0B10E8
 P 5950 3000
-F 0 "#PWR014" H 5950 2750 50  0001 C CNN
+F 0 "#PWR082" H 5950 2750 50  0001 C CNN
 F 1 "GND" H 5955 2827 50  0000 C CNN
 F 2 "" H 5950 3000 50  0001 C CNN
@@
 NoConn ~ 5500 4300
 $Comp
-L power:GND #PWR06
+L power:GND #PWR078
 U 1 1 5D81CFF2
 P 2650 5550
-F 0 "#PWR06" H 2650 5300 50  0001 C CNN
+F 0 "#PWR078" H 2650 5300 50  0001 C CNN
 F 1 "GND" H 2655 5377 50  0000 C CNN
 F 2 "" H 2650 5550 50  0001 C CNN
@@
 NoConn ~ 3250 3850
 $Comp
-L Connector:USB_C_Receptacle_USB2.0V1 J1
+L Connector:USB_C_Receptacle_USB2.0V1 J6
 U 1 1 5DAA54CA
 P 2650 3250
-F 0 "J1" H 2757 4117 50  0000 C CNN
+F 0 "J6" H 2757 4117 50  0000 C CNN
 F 1 "USB_C_Receptacle_USB2.0V1" H 2757 4026 50  0000 C CNN
 F 2 "Connector_USB:TYPE-C-31-M-12" H 2800 3250 50  0001 C CNN
@@
 Text HLabel 8950 3500 2    50   Input ~ 0
 TX
-Text HLabel 8950 3800 2    50   Input ~ 0
+Text HLabel 9600 3800 2    50   Input ~ 0
 ~Reset
+$Comp
+L Switch:SW_Push SW2
+U 1 1 5E0DEBC6
+P 9250 4650
+F 0 "SW2" V 9204 4798 50  0000 L CNN
+F 1 "SW_Push" V 9295 4798 50  0000 L CNN
+F 2 "Button_Switch_SMD:SW_SPST_PTS645" H 9250 4850 50  0001 C CNN
+F 3 "" H 9250 4850 50  0001 C CNN
+	1    9250 4650
+	0    1    1    0
+$EndComp
+$Comp
+L power:GND #PWR088
+U 1 1 5E0DF425
+P 9250 5550
+F 0 "#PWR088" H 9250 5300 50  0001 C CNN
+F 1 "GND" H 9255 5377 50  0000 C CNN
+F 2 "" H 9250 5550 50  0001 C CNN
+F 3 "" H 9250 5550 50  0001 C CNN
+	1    9250 5550
+	1    0    0    -1
+$EndComp
+Wire Wire Line
+	9250 5550 9250 4850
+Wire Wire Line
+	9250 4450 9250 3800
+Connection ~ 9250 3800
+Wire Wire Line
+	9250 3800 9600 3800
 $EndSCHEMATC

Commit message: radio hub board started
Parts:
- J6: symbol Connector:USB_C_Receptacle_USB2.0V1 -> radioDev-rescue:USB_C_Receptacle_USB2.0V1-Connector
- U11: symbol Interface_USB:FT232RL -> radioDev-rescue:FT232RL-Interface_USB
Changed lines of the file:
@@
 EESchema Schematic File Version 4
-LIBS:radioDev-cache
 EELAYER 30 0
 EELAYER END
@@
 $EndComp
 $Comp
-L Interface_USB:FT232RL U11
+L radioDev-rescue:FT232RL-Interface_USB U11
 U 1 1 5E0B10D6
 P 6300 4100
@@
 NoConn ~ 3250 3850
 $Comp
-L Connector:USB_C_Receptacle_USB2.0V1 J6
+L radioDev-rescue:USB_C_Receptacle_USB2.0V1-Connector J6
 U 1 1 5DAA54CA
 P 2650 3250
