File: hardware/radio_dev_board/devInt.sch (KiCad schematic (older format))
At the start: 10 parts

Commit message: added radio USB serial channel. Update board layout
Parts:
- C10, C11, C12, C9: renamed from C?; footprint (none) -> Capacitor_SMD:C_0603_1608Metric_Pad1.05x0.95mm_HandSolder
- J2, J3: renamed from J?; footprint (none) -> Connector_PinHeader_2.54mm:PinHeader_1x05_P2.54mm_Vertical
- U5, U6, U7, U8: renamed from U?; footprint (none) -> Package_SO:SSO-8_6.8x5.9mm_P1.27mm_Clearance7mm
Changed lines of the file:
@@
 $Descr A4 11693 8268
 encoding utf-8
-Sheet 3 5
+Sheet 3 6
 Title ""
 Date ""
@@
 $EndDescr
 $Comp
-L Interface:DS90LV028 U?
+L Interface:DS90LV028 U5
 U 1 1 5DCA47D4
 P 4650 1500
-F 0 "U?" H 4650 2281 50  0000 C CNN
+F 0 "U5" H 4650 2281 50  0000 C CNN
 F 1 "DS90LV028" H 4650 2190 50  0000 C CNN
-F 2 "" H 4650 1500 50  0001 C CNN
+F 2 "Package_SO:SSO-8_6.8x5.9mm_P1.27mm_Clearance7mm" H 4650 1500 50  0001 C CNN
 F 3 "" H 4650 1500 50  0001 C CNN
 	1    4650 1500
@@
 $EndComp
 $Comp
-L Interface:DS90LV028 U?
+L Interface:DS90LV028 U6
 U 1 1 5DCA48AA
 P 4650 3250
-F 0 "U?" H 4650 4031 50  0000 C CNN
+F 0 "U6" H 4650 4031 50  0000 C CNN
 F 1 "DS90LV028" H 4650 3940 50  0000 C CNN
-F 2 "" H 4650 3250 50  0001 C CNN
+F 2 "Package_SO:SSO-8_6.8x5.9mm_P1.27mm_Clearance7mm" H 4650 3250 50  0001 C CNN
 F 3 "" H 4650 3250 50  0001 C CNN
 	1    4650 3250
@@
 $EndComp
 $Comp
-L Interface:DS90LV028 U?
+L Interface:DS90LV028 U7
 U 1 1 5DCA5170
 P 4650 5000
-F 0 "U?" H 4650 5781 50  0000 C CNN
+F 0 "U7" H 4650 5781 50  0000 C CNN
 F 1 "DS90LV028" H 4650 5690 50  0000 C CNN
-F 2 "" H 4650 5000 50  0001 C CNN
+F 2 "Package_SO:SSO-8_6.8x5.9mm_P1.27mm_Clearance7mm" H 4650 5000 50  0001 C CNN
 F 3 "" H 4650 5000 50  0001 C CNN
 	1    4650 5000
@@
 $EndComp
 $Comp
-L Interface:DS90LV028 U?
+L Interface:DS90LV028 U8
 U 1 1 5DCA57CE
 P 4650 6750
-F 0 "U?" H 4650 7531 50  0000 C CNN
+F 0 "U8" H 4650 7531 50  0000 C CNN
 F 1 "DS90LV028" H 4650 7440 50  0000 C CNN
-F 2 "" H 4650 6750 50  0001 C CNN
+F 2 "Package_SO:SSO-8_6.8x5.9mm_P1.27mm_Clearance7mm" H 4650 6750 50  0001 C CNN
 F 3 "" H 4650 6750 50  0001 C CNN
 	1    4650 6750
@@
 $EndComp
 $Comp
-L power:+3.3V #PWR?
+L power:+3.3V #PWR027
 U 1 1 5DCA66B5
 P 3900 750
-F 0 "#PWR?" H 3900 600 50  0001 C CNN
+F 0 "#PWR027" H 3900 600 50  0001 C CNN
 F 1 "+3.3V" H 3915 923 50  0000 C CNN
 F 2 "" H 3900 750 50  0001 C CNN
@@
 $EndComp
 $Comp
-L power:GND #PWR?
+L power:GND #PWR035
 U 1 1 5DCA7509
 P 5250 6300
-F 0 "#PWR?" H 5250 6050 50  0001 C CNN
+F 0 "#PWR035" H 5250 6050 50  0001 C CNN
 F 1 "GND" H 5255 6127 50  0000 C CNN
 F 2 "" H 5250 6300 50  0001 C CNN
@@
 $EndComp
 $Comp
-L Device:C C?
+L Device:C C12
 U 1 1 5DCA7657
 P 5250 6100
-F 0 "C?" H 5365 6146 50  0000 L CNN
+F 0 "C12" H 5365 6146 50  0000 L CNN
 F 1 "C" H 5365 6055 50  0000 L CNN
-F 2 "" H 5288 5950 50  0001 C CNN
+F 2 "Capacitor_SMD:C_0603_1608Metric_Pad1.05x0.95mm_HandSolder" H 5288 5950 50  0001 C CNN
 F 3 "~" H 5250 6100 50  0001 C CNN
 	1    5250 6100
@@
 $EndComp
 $Comp
-L Device:C C?
+L Device:C C11
 U 1 1 5DCA8C03
 P 5250 4350
-F 0 "C?" H 5365 4396 50  0000 L CNN
+F 0 "C11" H 5365 4396 50  0000 L CNN
 F 1 "C" H 5365 4305 50  0000 L CNN
-F 2 "" H 5288 4200 50  0001 C CNN
+F 2 "Capacitor_SMD:C_0603_1608Metric_Pad1.05x0.95mm_HandSolder" H 5288 4200 50  0001 C CNN
 F 3 "~" H 5250 4350 50  0001 C CNN
 	1    5250 4350
@@
 $EndComp
 $Comp
-L Device:C C?
+L Device:C C10
 U 1 1 5DCA9176
 P 5250 2600
-F 0 "C?" H 5365 2646 50  0000 L CNN
+F 0 "C10" H 5365 2646 50  0000 L CNN
 F 1 "C" H 5365 2555 50  0000 L CNN
-F 2 "" H 5288 2450 50  0001 C CNN
+F 2 "Capacitor_SMD:C_0603_1608Metric_Pad1.05x0.95mm_HandSolder" H 5288 2450 50  0001 C CNN
 F 3 "~" H 5250 2600 50  0001 C CNN
 	1    5250 2600
@@
 $EndComp
 $Comp
-L Device:C C?
+L Device:C C9
 U 1 1 5DCAB2C5
 P 5250 850
-F 0 "C?" H 5365 896 50  0000 L CNN
+F 0 "C9" H 5365 896 50  0000 L CNN
 F 1 "C" H 5365 805 50  0000 L CNN
-F 2 "" H 5288 700 50  0001 C CNN
+F 2 "Capacitor_SMD:C_0603_1608Metric_Pad1.05x0.95mm_HandSolder" H 5288 700 50  0001 C CNN
 F 3 "~" H 5250 850 50  0001 C CNN
 	1    5250 850
@@
 $EndComp
 $Comp
-L power:GND #PWR?
+L power:GND #PWR034
 U 1 1 5DCAFF8D
 P 5250 4550
-F 0 "#PWR?" H 5250 4300 50  0001 C CNN
+F 0 "#PWR034" H 5250 4300 50  0001 C CNN
 F 1 "GND" H 5255 4377 50  0000 C CNN
 F 2 "" H 5250 4550 50  0001 C CNN
@@
 $EndComp
 $Comp
-L power:GND #PWR?
+L power:GND #PWR033
 U 1 1 5DCB180C
 P 5250 2800
-F 0 "#PWR?" H 5250 2550 50  0001 C CNN
+F 0 "#PWR033" H 5250 2550 50  0001 C CNN
 F 1 "GND" H 5255 2627 50  0000 C CNN
 F 2 "" H 5250 2800 50  0001 C CNN
@@
 $EndComp
 $Comp
-L power:GND #PWR?
+L power:GND #PWR028
 U 1 1 5DCB20B9
 P 4650 2200
-F 0 "#PWR?" H 4650 1950 50  0001 C CNN
+F 0 "#PWR028" H 4650 1950 50  0001 C CNN
 F 1 "GND" H 4655 2027 50  0000 C CNN
 F 2 "" H 4650 2200 50  0001 C CNN
@@
 $EndComp
 $Comp
-L power:GND #PWR?
+L power:GND #PWR031
 U 1 1 5DCB43F7
 P 4650 7450
-F 0 "#PWR?" H 4650 7200 50  0001 C CNN
+F 0 "#PWR031" H 4650 7200 50  0001 C CNN
 F 1 "GND" H 4655 7277 50  0000 C CNN
 F 2 "" H 4650 7450 50  0001 C CNN
@@
 $EndComp
 $Comp
-L power:GND #PWR?
+L power:GND #PWR030
 U 1 1 5DCB4808
 P 4650 5700
-F 0 "#PWR?" H 4650 5450 50  0001 C CNN
+F 0 "#PWR030" H 4650 5450 50  0001 C CNN
 F 1 "GND" H 4655 5527 50  0000 C CNN
 F 2 "" H 4650 5700 50  0001 C CNN
@@
 $EndComp
 $Comp
-L power:GND #PWR?
+L power:GND #PWR029
 U 1 1 5DCB6D60
 P 4650 3950
-F 0 "#PWR?" H 4650 3700 50  0001 C CNN
+F 0 "#PWR029" H 4650 3700 50  0001 C CNN
 F 1 "GND" H 4655 3777 50  0000 C CNN
 F 2 "" H 4650 3950 50  0001 C CNN
@@
 $EndComp
 $Comp
-L power:GND #PWR?
+L power:GND #PWR032
 U 1 1 5DCC6DCB
 P 5250 1050
-F 0 "#PWR?" H 5250 800 50  0001 C CNN
+F 0 "#PWR032" H 5250 800 50  0001 C CNN
 F 1 "GND" H 5255 877 50  0000 C CNN
 F 2 "" H 5250 1050 50  0001 C CNN
@@
 Connection ~ 4650 6150
 $Comp
-L Connector_Generic:Conn_01x05 J?
+L Connector_Generic:Conn_01x05 J3
 U 1 1 5DCD20C4
 P 6450 5850
-F 0 "J?" H 6530 5892 50  0000 L CNN
+F 0 "J3" H 6530 5892 50  0000 L CNN
 F 1 "Conn_01x05" H 6530 5801 50  0000 L CNN
-F 2 "" H 6450 5850 50  0001 C CNN
+F 2 "Connector_PinHeader_2.54mm:PinHeader_1x05_P2.54mm_Vertical" H 6450 5850 50  0001 C CNN
 F 3 "~" H 6450 5850 50  0001 C CNN
 	1    6450 5850
@@
 $EndComp
 $Comp
-L power:GND #PWR?
+L power:GND #PWR037
 U 1 1 5DCD28C2
 P 6100 6300
-F 0 "#PWR?" H 6100 6050 50  0001 C CNN
+F 0 "#PWR037" H 6100 6050 50  0001 C CNN
 F 1 "GND" H 6105 6127 50  0000 C CNN
 F 2 "" H 6100 6300 50  0001 C CNN
@@
 	5900 4800 5150 4800
 $Comp
-L Connector_Generic:Conn_01x05 J?
+L Connector_Generic:Conn_01x05 J2
 U 1 1 5DCD56C5
 P 6450 2350
-F 0 "J?" H 6530 2392 50  0000 L CNN
+F 0 "J2" H 6530 2392 50  0000 L CNN
 F 1 "Conn_01x05" H 6530 2301 50  0000 L CNN
-F 2 "" H 6450 2350 50  0001 C CNN
+F 2 "Connector_PinHeader_2.54mm:PinHeader_1x05_P2.54mm_Vertical" H 6450 2350 50  0001 C CNN
 F 3 "~" H 6450 2350 50  0001 C CNN
 	1    6450 2350
@@
 $EndComp
 $Comp
-L power:GND #PWR?
+L power:GND #PWR036
 U 1 1 5DCD7682
 P 6100 2800
-F 0 "#PWR?" H 6100 2550 50  0001 C CNN
+F 0 "#PWR036" H 6100 2550 50  0001 C CNN
 F 1 "GND" H 6105 2627 50  0000 C CNN
 F 2 "" H 6100 2800 50  0001 C CNN

Commit message: radio hub board started
Parts:
- U5, U6, U7, U8: symbol Interface:DS90LV028 -> radioDev-rescue:DS90LV028-Interface
Changed lines of the file:
@@
 EESchema Schematic File Version 4
-LIBS:radioDev-cache
 EELAYER 30 0
 EELAYER END
@@
 $EndDescr
 $Comp
-L Interface:DS90LV028 U5
+L radioDev-rescue:DS90LV028-Interface U5
 U 1 1 5DCA47D4
 P 4650 1500
@@
 $EndComp
 $Comp
-L Interface:DS90LV028 U6
+L radioDev-rescue:DS90LV028-Interface U6
 U 1 1 5DCA48AA
 P 4650 3250
@@
 $EndComp
 $Comp
-L Interface:DS90LV028 U7
+L radioDev-rescue:DS90LV028-Interface U7
 U 1 1 5DCA5170
 P 4650 5000
@@
 $EndComp
 $Comp
-L Interface:DS90LV028 U8
+L radioDev-rescue:DS90LV028-Interface U8
 U 1 1 5DCA57CE
 P 4650 6750
