File: hardware/radio_dev_board/devPSU.sch (KiCad schematic (older format))
At the start: 17 parts

Commit message: added radio USB serial channel. Update board layout
Parts:
- added C23, C26: 10u, Capacitor_THT:CP_Radial_D12.5mm_P5.00mm, symbol Device:CP
- added C24, C25: 0.1, Capacitor_SMD:C_0603_1608Metric_Pad1.05x0.95mm_HandSolder, symbol Device:C
- added D11, D12: D_Schottky, Diode_SMD:D_SOD-123F, symbol Device:D_Schottky
- added J5: Barrel_Jack_MountingPin, Connector_BarrelJack:BarrelJack_Wuerth_6941xx301002, symbol Connector:Barrel_Jack_Switch
- added U10: 78M05_Switcher, Package_TO_SOT_THT:TO-220-3_Vertical, symbol Regulator_Linear:LM78M05_TO220
- C16, C19: renamed from C?; footprint (none) -> Capacitor_SMD:C_1210_3225Metric_Pad1.42x2.65mm_HandSolder
- C17, C18: renamed from C?; footprint (none) -> Capacitor_SMD:C_0603_1608Metric_Pad1.05x0.95mm_HandSolder
- U9: renamed from U?; footprint (none) -> Package_TO_SOT_SMD:SOT-223-3_TabPin2
- gave numbers to parts that had none: 12
Connections:
- net +5V: now also D12.1 (K)
- net GND: now also C23.2, C24.2, C25.2, C26.2, J5.2, J5.3, U10.2 (GND)
- new net: C23.1, C24.1, D11.1 (K), J5.1, U10.1 (VI)
- new net: C25.1, C26.1, D11.2 (A), D12.2 (A), U10.3 (VO)

Commit message: added program and misc buttons. Finish layout
Parts:
- renumbered C23 to C13, C24 to C14, C13 to C15, C14 to C16, C15 to C17, C25 to C18, C26 to C19, C16 to C20, C17 to C21, C18 to C22, C19 to C23, D12 to D10, D5 to D11, D6 to D12, D11 to D8, D4 to D9, R10 to R14, R11 to R15, R12 to R16, R13 to R17, U9 to U10, U10 to U9

Commit message: radio hub board started
Parts:
- J4: symbol Connector:USB_C_Receptacle_USB2.0V1 -> radioDev-rescue:USB_C_Receptacle_USB2.0V1-Connector
Changed lines of the file:
@@
 EESchema Schematic File Version 4
-LIBS:radioDev-cache
 EELAYER 30 0
 EELAYER END
@@
 NoConn ~ 3900 4000
 $Comp
-L Connector:USB_C_Receptacle_USB2.0V1 J?
+L radioDev-rescue:USB_C_Receptacle_USB2.0V1-Connector J?
 U 1 1 5DCFE330
 P 3300 3400
 AR Path="/5DCC82D4/5DCFE330" Ref="J?"  Part="1"
 AR Path="/5DCCA0EA/5DCFE330" Ref="J4"  Part="1"
+AR Path="/5DCFE330" Ref="J4"  Part="1"
 F 0 "J4" H 3407 4267 50  0000 C CNN
 F 1 "USB_C_Receptacle_USB2.0V1" H 3407 4176 50  0000 C CNN
