File: hardware/radio_dev_board/radioDev.sch (KiCad schematic (older format))
At the start: 11 parts, among them J1 Conn_02x03_Odd_Even, U1 SP3485CN, U2 conn2x18pcie

Commit message: added program and misc buttons. Finish layout
Connections:
- wire segments 121 -> 120
Changed lines of the file:
@@
 F18 "D+" I L 2400 2450 50
 F19 "D-" I L 2400 2550 50
-F20 "~Reset~_Local" I L 2400 2200 50
 $EndSheet
 $Comp
@@
 	3950 2650 5000 2650
 Wire Wire Line
-	2400 2200 1550 2200
-Wire Wire Line
 	2400 2100 1550 2100
 Wire Wire Line
@@
 Text Label 1750 2100 0    50   ~ 0
 SCK
-Text Label 1750 2200 0    50   ~ 0
-~Reset
 Text Label 9000 5900 0    50   ~ 0
 MOSI
@@
 $EndComp
 Wire Wire Line
-	2450 1750 1550 1750
+	2400 1750 1550 1750
 Wire Wire Line
 	2400 1650 1550 1650

Commit message: radio hub board started
Parts:
- U2: symbol pcie:conn2x18pcie -> radioDev-rescue:conn2x18pcie-pcie
Changed lines of the file:
@@
 EESchema Schematic File Version 4
-LIBS:radioDev-cache
 EELAYER 30 0
 EELAYER END
@@
 $EndSheet
 $Comp
-L pcie:conn2x18pcie U2
+L radioDev-rescue:conn2x18pcie-pcie U2
 U 1 1 5DCC86DA
 P 8400 3300
