File: hardware/hub_module/optical.sch (KiCad schematic (older format))
At the start: 0 parts

Commit message: busses added
Parts:
- added C25, C27: 22u, symbol Device:C
- added C26, C28: 0.1u, symbol Device:C
- added J2: SFP+, Connector:Connector_SFP_and_Cage, symbol Interface_Optical:SFP+
- added JP217: Hi-Lo BW, symbol Device:Jumper_NO_Small
- added JP218: Hi-Low BW, symbol Device:Jumper_NO_Small
- added L1, L2: 4.7uH, symbol Device:L
- added R2, R3, R4, R5, R6, R7: 4k7, symbol Device:R
Connections:
- new net: C28.2, J2.15 (VccR)
- new net: C25.2, C26.2, C27.2, J2.16 (VccT)
- new net: J2.7 (RS0), JP217.1, R2.2
- new net: J2.9 (RS1), JP218.1, R3.2
- new net: C28.1, L2.2
- new net: C25.1, C26.1, C27.1, L1.2
- new net +3V3: L1.1, L2.1, R2.1, R3.1, R4.1, R5.1, R6.1, R7.1
- new net GND: J2.1 (VeeT), J2.10 (VeeR), J2.11 (VeeR), J2.14 (VeeR), J2.17 (VeeT), J2.20 (VeeT), J2.CAGE, JP217.2, JP218.2
- new net MOD-ABS: J2.6 (MOD_ABS), R5.2
- new net RD+: J2.13 (RD+)
- new net RD-: J2.12 (RD-)
- new net RX-LOS: J2.8 (RX_LOS), R7.2
- new net SFC-IIC-SCL: J2.5 (SCL)
- new net SFC-IIC-SDA: J2.4 (SDA)
- new net TD+: J2.18 (TD+)
- new net TD-: J2.19 (TD-)
- new net TX-DISABLE: J2.3 (TX_DISABLE), R4.2
- new net TX-FAULT: J2.2 (TX_FAULT), R6.2
